File: _autosave-ai03-pcb-guide.kicad_pcb (KiCad board)
At the start: 2 copper layers, 75.4 x 38.1 mm, 24 parts, among them SW1 SW_Push, U1 ATmega32U4-AU, Y1 16MHz

Commit message: Completed pcb design
Routing:
- added copper zone on F.Cu, net GND
Changed lines of the file:
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@@
   (segment (start 158.907 67.153) (end 160.401 67.153) (width 0.25) (layer F.Cu) (net 20))
   (segment (start 158.432 67.628) (end 158.907 67.153) (width 0.25) (layer F.Cu) (net 20))
+  (zone (net 1) (net_name GND) (layer F.Cu) (hatch edge 0.508)
+    (connect_pads (clearance 0.508))
+    (min_thickness 0.254)
+    (fill yes (arc_segments 32) (thermal_gap 0.508) (thermal_bridge_width 0.508))
+    (polygon
+      (pts
+        (xy 200.914 90.551) (xy 125.349 90.424) (xy 125.349 52.451) (xy 200.914 52.324)
+      )
+    )
+  )
 )
